File: geolight_sensorModule.sch (KiCad schematic (older format))
At the start: 18 parts, among them IC1 ATTINY841-SSU, P1 OPEN, P2 OPEN, P3 Male Pin Header, Angled (90*), P4 Male Pin Header, Angled (90*), P5 OPEN, P6 OPEN, U1 TCRT5000/L, Y1 16Mhz

Commit message: 90% complete for 8mm LED. Stopping for change back to 5mm.
Parts:
- JP1: value OPEN -> I2C/SPI
- JP2: value OPEN -> MISO_EN
- P1: value OPEN -> 5V inject
- P3: value Male Pin Header, Angled (90*) -> IN
- P4: value Male Pin Header, Angled (90*) -> OUT
- P5: value OPEN -> AUX Sensor
- P6: value OPEN -> DEBUG
Connections:
- net SCK/SCL: now also P4.4 (P4); no longer P4.1 (P1)
- net at JP1.2 (G2): now also P4.1 (P1); no longer P4.4 (P4)
Other:
- moved on the sheet: P4
Changed lines of the file:
@@
 P 3250 2600
 F 0 "P1" H 3250 2450 50  0000 C CNN
-F 1 "OPEN" H 3250 2750 50  0000 C CNN
+F 1 "5V inject" H 3250 2750 50  0000 C CNN
 F 2 "Terminal_Blocks:TerminalBlock_Pheonix_MPT-2.54mm_2pol" H 3250 2600 50  0001 C CNN
 F 3 "" H 3250 2600 50  0001 C CNN
@@
 P 6800 4500
 F 0 "P3" H 6800 4850 50  0000 C CNN
-F 1 "Male Pin Header, Angled (90*)" V 6900 4500 50  0000 C CNN
+F 1 "IN" V 6900 4500 50  0000 C CNN
 F 2 "Pin_Headers:Pin_Header_Straight_1x06" H 6800 4500 50  0001 C CNN
 F 3 "" H 6800 4500 50  0001 C CNN
@@
 L CONN_01X06 P4
 U 1 1 57CBE474
-P 9800 3850
-F 0 "P4" H 9800 4200 50  0000 C CNN
-F 1 "Male Pin Header, Angled (90*)" V 9900 3850 50  0000 C CNN
-F 2 "Pin_Headers:Pin_Header_Straight_1x06" H 9800 3850 50  0001 C CNN
-F 3 "" H 9800 3850 50  0001 C CNN
-F 4 "" H 0   0   50  0001 C CNN "MFR"
-F 5 "" H 0   0   50  0001 C CNN "MPN"
-F 6 "" H 0   0   50  0001 C CNN "SPR"
-F 7 "" H 0   0   50  0001 C CNN "SPN"
-F 8 "" H 0   0   50  0001 C CNN "SPURL"
-	1    9800 3850
+P 9800 3750
+F 0 "P4" H 9800 4100 50  0000 C CNN
+F 1 "OUT" V 9900 3750 50  0000 C CNN
+F 2 "Pin_Headers:Pin_Header_Straight_1x06" H 9800 3750 50  0001 C CNN
+F 3 "" H 9800 3750 50  0001 C CNN
+F 4 "" H 0   -100 50  0001 C CNN "MFR"
+F 5 "" H 0   -100 50  0001 C CNN "MPN"
+F 6 "" H 0   -100 50  0001 C CNN "SPR"
+F 7 "" H 0   -100 50  0001 C CNN "SPN"
+F 8 "" H 0   -100 50  0001 C CNN "SPURL"
+	1    9800 3750
 	1    0    0    -1
 $EndComp
@@
 P 5650 3550
 F 0 "P6" H 5750 3600 50  0000 C CNN
-F 1 "OPEN" H 5800 3500 50  0000 C CNN
+F 1 "DEBUG" H 5850 3500 50  0000 C CNN
 F 2 "Measurement_Points:Test_Point" H 5650 3550 50  0001 C CNN
 F 3 "" H 5650 3550 50  0001 C CNN
@@
 P 8200 4000
 F 0 "JP1" H 8150 4250 50  0000 C CNN
-F 1 "OPEN" H 8200 3800 50  0000 C CNN
+F 1 "I2C/SPI" H 8200 3800 50  0000 C CNN
 F 2 "Connect:GS3" V 8288 3926 50  0001 C CNN
 F 3 "" H 8200 4000 50  0001 C CNN
@@
 U 1 1 57CC1D1D
 P 8750 3900
-F 0 "JP2" V 8550 3750 50  0000 C CNN
-F 1 "OPEN" V 8650 3850 50  0000 C CNN
+F 0 "JP2" V 8950 3750 50  0000 C CNN
+F 1 "MISO_EN" V 9050 3850 50  0000 C CNN
 F 2 "Connect:GS2" V 8824 3900 50  0001 C CNN
 F 3 "" H 8750 3900 50  0001 C CNN
@@
 P 9800 2550
 F 0 "P5" H 9800 2750 50  0000 C CNN
-F 1 "OPEN" V 9900 2550 50  0000 C CNN
+F 1 "AUX Sensor" V 9900 2550 50  0000 C CNN
 F 2 "Pin_Headers:Pin_Header_Straight_1x03" H 9800 2550 50  0001 C CNN
 F 3 "" H 9800 2550 50  0001 C CNN
@@
 Text Label 5300 3600 0    60   ~ 0
 RX
-Text Label 9050 3600 0    60   ~ 0
+Text Label 9000 3800 0    60   ~ 0
 SCK/SCL
 Text Label 7550 3900 0    60   ~ 0
 MISO
-Text Label 9050 4100 0    60   ~ 0
+Text Label 9000 4000 0    60   ~ 0
 SS
 Text Label 1050 2550 0    60   ~ 0
@@
 	8050 4100 8200 4100
 Wire Wire Line
-	9600 4100 9050 4100
+	9200 4000 9000 4000
 Wire Wire Line
 	5850 2900 6300 2900
@@
 	3150 4300 3000 4300
 Wire Wire Line
-	3450 2650 3450 2650
-Wire Wire Line
-	3650 2650 3450 2650
-Wire Wire Line
-	3450 2550 3450 2550
-Wire Wire Line
-	3650 2550 3450 2550
+	3450 2650 3650 2650
+Wire Wire Line
+	3450 2550 3650 2550
 Wire Wire Line
 	3650 2650 3650 2900
 Wire Wire Line
-	3650 2300 3650 2550
+	3650 2550 3650 2300
 Wire Wire Line
 	5800 4600 5800 4900
@@
 	6250 4200 6250 4300
 Wire Wire Line
-	9600 3600 9050 3600
-Wire Wire Line
-	9600 3700 9500 3700
-Wire Wire Line
-	9500 3700 9500 3450
-Wire Wire Line
-	9600 3800 9500 3800
-Wire Wire Line
-	9500 3800 9500 4200
-Wire Wire Line
-	8950 3900 9200 3900
-Wire Wire Line
-	9200 3900 9400 4000
+	9500 3700 9500 4200
+Wire Wire Line
+	8950 3900 9600 3900
+Wire Wire Line
+	8350 4000 8500 4000
+Wire Wire Line
+	9200 4000 9400 4000
 Wire Wire Line
 	9400 4000 9600 4000
 Wire Wire Line
-	8350 4000 9200 4000
-Wire Wire Line
-	9200 4000 9400 3900
-Wire Wire Line
-	9400 3900 9600 3900
+	9500 3450 9500 3600
+Wire Wire Line
+	9500 3600 9600 3600
+Wire Wire Line
+	9500 3700 9600 3700
+Wire Wire Line
+	8500 4000 8500 3500
+Wire Wire Line
+	8500 3500 9600 3500
+Wire Wire Line
+	9600 3800 9000 3800
 $EndSCHEMATC

Commit message: 5mm, rev2 stage (wait a day and finalize)
Connections:
- net SDA/MOSI: now also JP1.2 (G2), P4.1 (P1)
Changed lines of the file:
@@
 	7550 4000 8050 4000
 Wire Wire Line
-	7550 3900 8050 3900
-Wire Wire Line
-	8050 3900 8550 3900
+	7550 3900 8550 3900
 Wire Wire Line
 	8200 4100 8200 4000
@@
 	8050 4100 8200 4100
 Wire Wire Line
-	9200 4000 9000 4000
+	9000 4000 9600 4000
 Wire Wire Line
-	5850 2900 6300 2900
-Wire Wire Line
-	6300 2900 6750 2900
+	5850 2900 6750 2900
 Wire Wire Line
 	4300 2700 4300 2800
@@
 	5900 2650 5850 2650
 Wire Wire Line
-	2500 4400 2500 4750
-Wire Wire Line
-	2500 4750 2500 4850
+	2500 4400 2500 4850
 Wire Wire Line
 	2750 4400 2500 4400
@@
 	2850 4200 2850 3900
 Wire Wire Line
-	2850 2300 2850 3400
-Wire Wire Line
-	2850 3400 2850 3700
+	2850 2300 2850 3700
 Wire Wire Line
 	4700 2800 4700 2700
@@
 	4700 2400 4700 2500
 Wire Wire Line
-	4300 2800 4500 2800
-Wire Wire Line
-	4500 2800 4700 2800
+	4300 2800 4700 2800
 Wire Wire Line
 	4500 2900 4500 2800
 Wire Wire Line
-	4300 2400 4500 2400
-Wire Wire Line
-	4500 2400 4700 2400
+	4300 2400 4700 2400
 Wire Wire Line
 	4500 2300 4500 2400
@@
 	5250 3600 5450 3600
 Wire Wire Line
-	5550 2350 5700 2350
-Wire Wire Line
-	5700 2350 5900 2350
+	5550 2350 5900 2350
 Wire Wire Line
 	5200 2300 5200 2350
@@
 	8950 3900 9600 3900
 Wire Wire Line
-	8350 4000 8500 4000
-Wire Wire Line
-	9200 4000 9400 4000
-Wire Wire Line
-	9400 4000 9600 4000
+	8200 4000 8500 4000
 Wire Wire Line
 	9500 3450 9500 3600
